Commit message: Joint limits updated

File: ur_description/urdf/ur5.urdf.xacro (robot description, xacro)
@@ -118,4 +118,5 @@
       </xacro:cylinder_inertial>
     </link>
+    <!-- Setting shoulder lift joint to -9 to -171 to never go below the table -->
     <joint name="${prefix}shoulder_lift_joint" type="revolute">
       <parent link="${prefix}shoulder_link" />
@@ -124,5 +125,5 @@
       <axis xyz="0 1 0" />
       <xacro:unless value="${joint_limited}">
-        <limit lower="${-2.0 * pi}" upper="${2.0 * pi}" effort="150.0" velocity="3.15"/>
+        <limit lower="${-19.0 * pi / 20.0}" upper="${-1.0 * pi / 20.0}" effort="150.0" velocity="3.15"/>
       </xacro:unless>
       <xacro:if value="${joint_limited}">
@@ -155,5 +156,5 @@
       <axis xyz="0 1 0" />
       <xacro:unless value="${joint_limited}">
-        <limit lower="${-2.0 * pi}" upper="${2.0 * pi}" effort="150.0" velocity="3.15"/>
+        <limit lower="${-8.0 * pi / 9.0}" upper="${8.0 * pi / 9.0}" effort="150.0" velocity="3.15"/>
       </xacro:unless>
       <xacro:if value="${joint_limited}">
@@ -306,4 +307,11 @@
       <child link="${prefix}tool0"/>
     </joint>
+    <!-- Frame coincident with all-zeros TCP on UR controller -->
+    <link name="${prefix}tool0_controller"/>
+    <joint name="${prefix}base_tool0_controller_floating_joint" type="floating">
+      <origin xyz="0 0 0" rpy="0 0 0"/>
+      <parent link="${prefix}base"/>
+      <child link="${prefix}tool0_controller"/>
+    </joint>
   </xacro:macro>
 </robot>
